File: trackix/trackix.sch (KiCad schematic (older format))
At the start: 42 parts, among them IC1 SIM808, J1 GSM, J2 GPS, J3 SIM5060-6-0-26-01-X_REVC, J4 AVR-ISP-6, Q1 2N3904, Q2 2N3904, U1 ATmega328P-AU

Commit message: layout changes 1
Parts:
- removed J3: SIM5060-6-0-26-01-X_REVC, SIM5060-6-0-26-01-X_REVC:GCT_SIM5060-6-0-26-01-X_REVC, symbol SIM5060-6-0-26-01-X_REVC:SIM5060-6-0-26-01-X_REVC
- added J3: SIM7100-6-1-15-00-X_REVA, SIM7100-6-1-15-00-X_REVA:GCT_SIM7100-6-1-15-00-X_REVA, symbol SIM7100-6-1-15-00-X_REVA:SIM7100-6-1-15-00-X_REVA
- 8MHz1: symbol Device:Crystal -> trackix-rescue:Crystal-Device
- BT1: symbol Device:Battery_Cell -> trackix-rescue:Battery_Cell-Device
- C10, C11, C12, C13, C14: symbol Device:C_Small -> trackix-rescue:C_Small-Device
- D1, D2, D3, D4, D5, D6: symbol Device:LED -> trackix-rescue:LED-Device
- IC1: symbol SIM808:SIM808 -> trackix-rescue:SIM808-SIM808
- J1, J2: symbol Connector:Conn_Coaxial -> trackix-rescue:Conn_Coaxial-Connector
- J4: symbol Connector:AVR-ISP-6 -> trackix-rescue:AVR-ISP-6-Connector
- JP1: symbol Device:Jumper_NC_Dual -> trackix-rescue:Jumper_NC_Dual-Device
- LS1: symbol CBT-09427-SMT:CBT-09427-SMT -> trackix-rescue:CBT-09427-SMT-CBT-09427-SMT
- Q1, Q2: symbol Transistor_BJT:2N3904 -> trackix-rescue:2N3904-Transistor_BJT
- R1, R2, R3, R4, R5, R6, R7, R8, R9: symbol Device:R -> trackix-rescue:R-Device
- U1: symbol MCU_Microchip_ATmega:ATmega328P-AU -> trackix-rescue:ATmega328P-AU-MCU_Microchip_ATmega
- reset1: symbol Switch:SW_Push -> trackix-rescue:SW_Push-Switch
Changed lines of the file:
@@
 $EndDescr
 $Comp
-L SIM808:SIM808 IC1
+L trackix-rescue:SIM808-SIM808 IC1
 U 1 1 5C6715B2
 P 2900 3900
@@
 	3950 5400 3700 5400
 $Comp
-L Device:R R3
+L trackix-rescue:R-Device R3
 U 1 1 5C67599C
 P 4700 5200
@@
 $EndComp
 $Comp
-L Device:R R2
+L trackix-rescue:R-Device R2
 U 1 1 5C675A49
 P 4700 5300
@@
 $EndComp
 $Comp
-L Device:R R1
+L trackix-rescue:R-Device R1
 U 1 1 5C675AC4
 P 4700 5600
@@
 $EndComp
 $Comp
-L Device:LED D1
+L trackix-rescue:LED-Device D1
 U 1 1 5C67E447
 P 4100 4500
@@
 $EndComp
 $Comp
-L Device:R R4
+L trackix-rescue:R-Device R4
 U 1 1 5C67E55B
 P 5000 4500
@@
 	2100 5500 1550 5500
 $Comp
-L Connector:Conn_Coaxial J2
+L trackix-rescue:Conn_Coaxial-Connector J2
 U 1 1 5C697DB2
 P 1550 4750
@@
 $EndComp
 $Comp
-L Connector:Conn_Coaxial J1
+L trackix-rescue:Conn_Coaxial-Connector J1
 U 1 1 5C697E95
 P 1100 4750
@@
 	1300 4750 1300 4900
 $Comp
-L MCU_Microchip_ATmega:ATmega328P-AU U1
+L trackix-rescue:ATmega328P-AU-MCU_Microchip_ATmega U1
 U 1 1 5C69F59F
 P 8650 3050
@@
 $EndComp
 $Comp
-L Device:Crystal 8MHz1
+L trackix-rescue:Crystal-Device 8MHz1
 U 1 1 5C69FEF1
 P 10350 2550
@@
 $EndComp
 $Comp
-L Device:C_Small C11
+L trackix-rescue:C_Small-Device C11
 U 1 1 5C6A0E74
 P 10800 2400
@@
 $EndComp
 $Comp
-L Device:C_Small C10
+L trackix-rescue:C_Small-Device C10
 U 1 1 5C6A0F45
 P 10800 2700
@@
 	8650 1400 8650 1550
 $Comp
-L Device:C_Small C12
+L trackix-rescue:C_Small-Device C12
 U 1 1 5C6B2906
 P 7850 1850
@@
 $EndComp
 $Comp
-L Device:R R6
+L trackix-rescue:R-Device R6
 U 1 1 5C6B93E2
 P 9650 3050
@@
 	9650 2800 9650 2900
 $Comp
-L Device:LED D2
+L trackix-rescue:LED-Device D2
 U 1 1 5C6C4882
 P 10350 1950
@@
 $EndComp
 $Comp
-L Device:R R7
+L trackix-rescue:R-Device R7
 U 1 1 5C6C4BDB
 P 9950 2150
@@
 	10600 1950 10600 2100
 $Comp
-L Connector:AVR-ISP-6 J4
+L trackix-rescue:AVR-ISP-6-Connector J4
 U 1 1 5C6CC941
 P 9950 1050
@@
 $EndComp
 $Comp
-L Device:Jumper_NC_Dual JP1
+L trackix-rescue:Jumper_NC_Dual-Device JP1
 U 1 1 5C6CCCFE
 P 11050 950
@@
 	11200 1350 11200 1300
 $Comp
-L Device:Battery_Cell BT1
+L trackix-rescue:Battery_Cell-Device BT1
 U 1 1 5C6D0064
 P 11750 950
@@
 $EndComp
 $Comp
-L Device:C_Small C14
+L trackix-rescue:C_Small-Device C14
 U 1 1 5C6EEA9E
 P 14650 1150
@@
 $EndComp
 $Comp
-L Device:C_Small C13
+L trackix-rescue:C_Small-Device C13
 U 1 1 5C70B4FC
 P 14250 1150
@@
 	1850 3600 2100 3600
 $Comp
-L Transistor_BJT:2N3904 Q1
+L trackix-rescue:2N3904-Transistor_BJT Q1
 U 1 1 5C72ED41
 P 10100 4650
@@
 $EndComp
 $Comp
-L Device:R R5
+L trackix-rescue:R-Device R5
 U 1 1 5C72EFB0
 P 9400 4450
@@
 	10200 4850 10200 5050
 $Comp
-L Transistor_BJT:2N3904 Q2
+L trackix-rescue:2N3904-Transistor_BJT Q2
 U 1 1 5C758481
 P 11650 4150
@@
 $EndComp
 $Comp
-L Device:R R9
+L trackix-rescue:R-Device R9
 U 1 1 5C75D87F
 P 11250 4150
@@
 	10200 3350 10300 3350
 $Comp
-L Switch:SW_Push reset1
+L trackix-rescue:SW_Push-Switch reset1
 U 1 1 5C6B6F4E
 P 10000 3350
@@
 	11750 4350 11750 4650
 $Comp
-L Device:LED D5
+L trackix-rescue:LED-Device D5
 U 1 1 5C78419F
 P 12050 3600
@@
 $EndComp
 $Comp
-L Device:LED D6
+L trackix-rescue:LED-Device D6
 U 1 1 5C7842CF
 P 12050 3800
@@
 $EndComp
 $Comp
-L Device:LED D4
+L trackix-rescue:LED-Device D4
 U 1 1 5C7898D9
 P 12050 3400
@@
 	9400 4250 9250 4250
 $Comp
-L Device:LED D3
+L trackix-rescue:LED-Device D3
 U 1 1 5C81A3A1
 P 10900 1550
@@
 $EndComp
 $Comp
-L Device:R R8
+L trackix-rescue:R-Device R8
 U 1 1 5C81AB5D
 P 10650 1200
@@
 	10750 1550 10650 1550
 $Comp
-L CBT-09427-SMT:CBT-09427-SMT LS1
+L trackix-rescue:CBT-09427-SMT-CBT-09427-SMT LS1
 U 1 1 5C851AE6
 P 10800 4900
@@
 	10400 5100 10800 5100
 $Comp
-L SIM5060-6-0-26-01-X_REVC:SIM5060-6-0-26-01-X_REVC J3
-U 1 1 5C862014
-P 5700 5350
-F 0 "J3" H 5700 5717 50  0000 C CNN
-F 1 "SIM5060-6-0-26-01-X_REVC" H 5700 5626 50  0000 C CNN
-F 2 "SIM5060-6-0-26-01-X_REVC:GCT_SIM5060-6-0-26-01-X_REVC" H 5700 5350 50  0001 L BNN
-F 3 "None" H 5700 5350 50  0001 L BNN
-F 4 "Unavailable" H 5700 5350 50  0001 L BNN "Field4"
-F 5 "Global Connector Technology" H 5700 5350 50  0001 L BNN "Field5"
-F 6 "SIM5060-6-0-26-01-A" H 5700 5350 50  0001 L BNN "Field6"
-F 7 "None" H 5700 5350 50  0001 L BNN "Field7"
-F 8 "6 Position 2.6 mm Profile Surface Mount Hinged SIM Card Connector" H 5700 5350 50  0001 L BNN "Field8"
-	1    5700 5350
-	1    0    0    -1
-$EndComp
-$Comp
 L power:GND #PWR0102
 U 1 1 5C86A9E8
-P 6250 5650
-F 0 "#PWR0102" H 6250 5400 50  0001 C CNN
-F 1 "GND" H 6255 5477 50  0000 C CNN
-F 2 "" H 6250 5650 50  0001 C CNN
-F 3 "" H 6250 5650 50  0001 C CNN
-	1    6250 5650
-	1    0    0    -1
-$EndComp
-Wire Wire Line
-	6100 5450 6250 5450
-Wire Wire Line
-	6250 5450 6250 5650
-Wire Wire Line
-	6100 5350 6300 5350
-Wire Wire Line
-	6300 5350 6300 5100
+P 6250 6250
+F 0 "#PWR0102" H 6250 6000 50  0001 C CNN
+F 1 "GND" H 6255 6077 50  0000 C CNN
+F 2 "" H 6250 6250 50  0001 C CNN
+F 3 "" H 6250 6250 50  0001 C CNN
+	1    6250 6250
+	1    0    0    -1
+$EndComp
 Wire Wire Line
 	4950 5100 6300 5100
 Wire Wire Line
-	5200 5200 5200 5250
-Wire Wire Line
-	5200 5250 5300 5250
-Wire Wire Line
-	4850 5200 5200 5200
-Wire Wire Line
-	5300 5350 5200 5350
-Wire Wire Line
-	5200 5350 5200 5600
-Wire Wire Line
 	4850 5600 5200 5600
-Wire Wire Line
-	5300 5450 5050 5450
-Wire Wire Line
-	5050 5450 5050 5300
+$Comp
+L SIM7100-6-1-15-00-X_REVA:SIM7100-6-1-15-00-X_REVA J3
+U 1 1 5C6B3FC2
+P 5700 6000
+F 0 "J3" H 5700 6367 50  0000 C CNN
+F 1 "SIM7100-6-1-15-00-X_REVA" H 5700 6276 50  0000 C CNN
+F 2 "SIM7100-6-1-15-00-X_REVA:GCT_SIM7100-6-1-15-00-X_REVA" H 5700 6000 50  0001 L BNN
+F 3 "None" H 5700 6000 50  0001 L BNN
+F 4 "Global Connector Technology" H 5700 6000 50  0001 L BNN "Field4"
+F 5 "None" H 5700 6000 50  0001 L BNN "Field5"
+F 6 "6 Position 2.54 mm Pitch Push-Push 1.5 mm Profile Micro SIM Card Connector" H 5700 6000 50  0001 L BNN "Field6"
+F 7 "SIM7100-6-1-15-00-A" H 5700 6000 50  0001 L BNN "Field7"
+F 8 "Unavailable" H 5700 6000 50  0001 L BNN "Field8"
+	1    5700 6000
+	1    0    0    -1
+$EndComp
+Wire Wire Line
+	6100 6100 6250 6100
+Wire Wire Line
+	6250 6100 6250 6250
+Wire Wire Line
+	6100 6000 6300 6000
+Wire Wire Line
+	5050 6100 5300 6100
+Wire Wire Line
+	5200 5600 5200 6000
+Wire Wire Line
+	5200 6000 5300 6000
+Wire Wire Line
+	5300 5900 5250 5900
+Wire Wire Line
+	5250 5900 5250 5200
+Wire Wire Line
+	4850 5200 5250 5200
+Wire Wire Line
+	5050 5300 5050 6100
+Wire Wire Line
+	6300 5100 6300 6000
 $EndSCHEMATC

Commit message: layout changes 2
Parts:
- added BR?: DB107S, DIOB_DB107S, symbol DB107S:DB107S
- added C?: 22pF, Capacitor_SMD:C_0805_2012Metric_Pad1.15x1.40mm_HandSolder, symbol trackix-rescue:C_Small-Device
- added D?: LED_chrg, LEDs:LED_0805_HandSoldering, symbol trackix-rescue:LED-Device
- added D?: LED_stdby, LEDs:LED_0805_HandSoldering, symbol trackix-rescue:LED-Device
- added H?: dynamo_A, symbol mechanical:MountingHole_Pad
- added H?: dynamo_B, symbol mechanical:MountingHole_Pad
- added IC?: TP4056, SOP-8, symbol TP4056:TP4056
- added Q?: FS8205A, SOP65P640X120-8N, symbol FS8205A:FS8205A
- added R10, R11, R12, R? (x2): 470, Resistors_SMD:R_0805_HandSoldering, symbol trackix-rescue:R-Device
- added U?: DW-01, SOT23-6, symbol DW-01:DW-01
- 8MHz1: footprint Crystal:Crystal_SMD_HC49-SD -> Crystals:Crystal_HC49-4H_Vertical
- D1, D2, D3: footprint LED_SMD:LED_0805_2012Metric_Pad1.15x1.40mm_HandSolder -> LEDs:LED_0805_HandSoldering
- D4, D5: footprint LED_THT:LED_D5.0mm_Horizontal_O6.35mm_Z15.0mm -> LEDs:LED_D5.0mm_Horizontal_O1.27mm_Z3.0mm
- D6: footprint LED_THT:LED_D5.0mm_FlatTop -> LEDs:LED_D5.0mm
- R1, R2, R3, R4, R5, R6, R7, R8, R9: footprint Resistor_SMD:R_0805_2012Metric_Pad1.15x1.40mm_HandSolder -> Resistors_SMD:R_0805_HandSoldering
- reset1: footprint Button_Switch_SMD:SW_SPST_TL3342 -> Buttons_Switches_SMD:SW_SPST_B3U-1000P
Connections:
- net labels added: AC, DYNAMO_A, DYNAMO_B, Earth
- wire segments 184 -> 226

Commit message: prototype 0.1 state
Parts:
- added C? (x2): 10uF, Capacitor_SMD:C_0805_2012Metric_Pad1.15x1.40mm_HandSolder, symbol trackix-rescue:C_Small-Device
- added C?: 0,1uF, Capacitor_SMD:C_0805_2012Metric_Pad1.15x1.40mm_HandSolder, symbol trackix-rescue:C_Small-Device
- added R15: 4k for Ibat 300mA, Resistors_SMD:R_0805_HandSoldering, symbol trackix-rescue:R-Device
- added R?: 100, Resistors_SMD:R_0805_HandSoldering, symbol trackix-rescue:R-Device
- added R?: 1k, Resistors_SMD:R_0805_HandSoldering, symbol trackix-rescue:R-Device
- added U2: SIM-ST-MFF2, SIM-ST-MFF2:PSON127P500X600X82-9N, symbol SIM-ST-MFF2:SIM-ST-MFF2
- gave numbers to parts that had none: 11
Connections:
- net labels added: -BATT
- net labels removed: AC, Earth
- wire segments 226 -> 276

Commit message: all things so far
Parts:
- removed BR1: DB107S, DIOB_DB107S, symbol DB107S:DB107S
- removed BT1: Li-Ion 3,7v, Connector_PinHeader_2.54mm:PinHeader_1x02_P2.54mm_Horizontal, symbol trackix-rescue:Battery_Cell-Device
- removed C1, C3, C4: 22pF, Capacitor_SMD:C_0805_2012Metric_Pad1.15x1.40mm_HandSolder, symbol pspice:CAP
- removed C12: 0,1uF, Capacitor_SMD:C_0805_2012Metric_Pad1.15x1.40mm_HandSolder, symbol trackix-rescue:C_Small-Device
- removed C2, C5: 1uF, Capacitor_Tantalum_SMD:CP_EIA-3216-10_Kemet-I_Pad1.58x1.35mm_HandSolder, symbol pspice:CAP
- removed C6: 100uF, Capacitor_Tantalum_SMD:CP_EIA-3216-10_Kemet-I_Pad1.58x1.35mm_HandSolder, symbol pspice:CAP
- removed C7: 10uF, Capacitor_Tantalum_SMD:CP_EIA-3216-10_Kemet-I_Pad1.58x1.35mm_HandSolder, symbol pspice:CAP
- removed C8: 33pF, Capacitor_SMD:C_0805_2012Metric_Pad1.15x1.40mm_HandSolder, symbol pspice:CAP
- removed C9: 10pF, Capacitor_SMD:C_0805_2012Metric_Pad1.15x1.40mm_HandSolder, symbol pspice:CAP
- removed C?: 10uF, Capacitor_SMD:C_0805_2012Metric_Pad1.15x1.40mm_HandSolder, symbol trackix-rescue:C_Small-Device
- removed D1: netstat LED, LEDs:LED_0805_HandSoldering, symbol trackix-rescue:LED-Device
- removed D3: ISP led, LEDs:LED_0805_HandSoldering, symbol trackix-rescue:LED-Device
- removed H1: dynamo_A, symbol mechanical:MountingHole_Pad
- removed H2: dynamo_B, symbol mechanical:MountingHole_Pad
- removed IC1: SIM808, SIM808:QFN100P2400X2400X260-68N, symbol trackix-rescue:SIM808-SIM808
- removed J1: GSM, Connector_Coaxial:U.FL_Hirose_U.FL-R-SMT-1_Vertical, symbol trackix-rescue:Conn_Coaxial-Connector
- removed J2: GPS, Connector_Coaxial:U.FL_Hirose_U.FL-R-SMT-1_Vertical, symbol trackix-rescue:Conn_Coaxial-Connector
- removed J3: SIM7100-6-1-15-00-X_REVA, SIM7100-6-1-15-00-X_REVA:GCT_SIM7100-6-1-15-00-X_REVA, symbol SIM7100-6-1-15-00-X_REVA:SIM7100-6-1-15-00-X_REVA
- removed JP1: Power Selector, Connector_PinSocket_2.54mm:PinSocket_1x03_P2.54mm_Vertical, symbol trackix-rescue:Jumper_NC_Dual-Device
- removed LS1: CBT-09427-SMT, CBT-09427-SMT:CUI_CBT-09427-SMT, symbol trackix-rescue:CBT-09427-SMT-CBT-09427-SMT
- removed Q2: 2N3904, Package_TO_SOT_SMD:SOT-23_Handsoldering, symbol trackix-rescue:2N3904-Transistor_BJT
- removed R1, R2, R3: 22, Resistors_SMD:R_0805_HandSoldering, symbol trackix-rescue:R-Device
- removed R4, R8: 470, Resistors_SMD:R_0805_HandSoldering, symbol trackix-rescue:R-Device
- removed U2: SIM-ST-MFF2, SIM-ST-MFF2:PSON127P500X600X82-9N, symbol SIM-ST-MFF2:SIM-ST-MFF2
- added BZ1: Buzzer, Buzzers_Beepers:Buzzer_Murata_PKMCS0909E4000-R1, symbol Device:Buzzer
- added C12, C2, C9: 10uF, Capacitors_SMD:C_1206, symbol trackix-rescue:C_Small-Device-trackix-rescue
- added C16, C8: 100nF, Capacitors_SMD:C_0603, symbol trackix-rescue:C_Small-Device-trackix-rescue
- added C17: C_100nF, Capacitors_SMD:C_0603, symbol trackix-rescue:C_Small-Device-trackix-rescue
- added C4, C6: C_4.7uF, Capacitors_SMD:C_1206, symbol Device:C
- added C5, C7: C_100nF, Capacitors_SMD:C_0603, symbol Device:C
- added D1: GPS_LED, LEDs:LED_0805, symbol trackix-rescue:LED-Device-trackix-rescue
- added D10, D11, D3, D9: D_B5818WS SK, Diodes_SMD:D_SOD-323, symbol Device:D
- added H1: DYNAMO_A, Mounting_Holes:MountingHole_2.2mm_M2_ISO14580_Pad, symbol Mechanical:MountingHole_Pad
- added H2: DYNAMO_B, Mounting_Holes:MountingHole_2.2mm_M2_ISO14580_Pad, symbol Mechanical:MountingHole_Pad
- added J1: BATTERY, Pin_Headers:Pin_Header_Straight_1x02_Pitch2.54mm, symbol Connector:Conn_01x02_Male
- added J2: GPS, Connectors_Molex:Molex_Microcoaxial_RF, symbol trackix-rescue:Conn_Coaxial-Connector-trackix-rescue
- added J3: LORA_868, Connectors_Molex:Molex_Microcoaxial_RF, symbol trackix-rescue:Conn_Coaxial-Connector-trackix-rescue
- added JP1: SCK, Jumper:SolderJumper-2_P1.3mm_Open_RoundedPad1.0x1.5mm, symbol Jumper:SolderJumper_2_Open
- added JP3: MOSI, Jumper:SolderJumper-2_P1.3mm_Open_RoundedPad1.0x1.5mm, symbol Jumper:SolderJumper_2_Open
- added JP4: MISO, Jumper:SolderJumper-2_P1.3mm_Open_RoundedPad1.0x1.5mm, symbol Jumper:SolderJumper_2_Open
- added L1: L27nH, Inductors_SMD:L_0402, symbol Device:L
- added L2: L2.2uH, Inductors_SMD:L_1210, symbol Device:L
- added Q5: 2N3904, TO_SOT_Packages_SMD:SOT-23, symbol trackix-rescue:2N3904-Transistor_BJT-trackix-rescue
- added R16, R18: R100, Resistors_SMD:R_0603, symbol device:R
- added R17: R22, Resistors_SMD:R_0603, symbol device:R
- added R19: R5k, Resistors_SMD:R_0603, symbol device:R
- added R20: R10k, Resistors_SMD:R_0603, symbol device:R
- added R21, R8: 4.7k, Resistors_SMD:R_0603, symbol trackix-rescue:R-Device-trackix-rescue
- added TP1: DYNAMO_A, Connectors_TestPoints:Test_Point_Pad_1.0x1.0mm, symbol Connector:TestPoint
- added TP2: DYNAMO_B, Connectors_TestPoints:Test_Point_Pad_1.0x1.0mm, symbol Connector:TestPoint
- added TP3: GND, Connectors_TestPoints:Test_Point_Pad_1.0x1.0mm, symbol Connector:TestPoint
- added TP4: VCC_IN_DC, Connectors_TestPoints:Test_Point_Pad_1.0x1.0mm, symbol Connector:TestPoint
- added TP5: AUX_ON, Connectors_TestPoints:Test_Point_Pad_1.0x1.0mm, symbol Connector:TestPoint
- added TP6: GPS_TX, Connectors_TestPoints:Test_Point_Pad_1.0x1.0mm, symbol Connector:TestPoint
- added TP7: TX, Connectors_TestPoints:Test_Point_Pad_1.0x1.0mm, symbol Connector:TestPoint
- added TP8: RX, Connectors_TestPoints:Test_Point_Pad_1.0x1.0mm, symbol Connector:TestPoint
- added TP9: TestPoint3.3V, Connectors_TestPoints:Test_Point_Pad_1.0x1.0mm, symbol Connector:TestPoint
- added U2: SIM28ML, SIM28ML:XCVR_SIM28ML, symbol RF_GPS:SIM28ML
- added U4: TPS62291DRVR, user_added_kicad_libs:SON65P200X200X80-7N, symbol TPS62291DRVR:TPS62291DRVR
- added U5: RFM95W-868S2, RF_Modules:Hopref_RFM9XW_SMD, symbol RF_Module:RFM95W-868S2
- added U6: ADXL345BCCZ, Housings_LGA:Bosch_LGA-14_3x2.5mm_Pitch0.5mm, symbol ADXL345BCCZ:ADXL345BCCZ
- 8MHz1: footprint Crystals:Crystal_HC49-4H_Vertical -> Crystals:Crystal_HC49-U_Vertical; symbol trackix-rescue:Crystal-Device -> trackix-rescue:Crystal-Device-trackix-rescue
- C1: renamed from C?; value 10uF -> 100nF; footprint Capacitor_SMD:C_0805_2012Metric_Pad1.15x1.40mm_HandSolder -> Capacitors_SMD:C_0805; symbol trackix-rescue:C_Small-Device -> trackix-rescue:C_Small-Device-trackix-rescue
- C10, C11: footprint Capacitor_SMD:C_0805_2012Metric_Pad1.15x1.40mm_HandSolder -> Capacitors_SMD:C_0402; symbol trackix-rescue:C_Small-Device -> trackix-rescue:C_Small-Device-trackix-rescue
- C13: footprint Capacitor_Tantalum_SMD:CP_EIA-3216-10_Kemet-I_Pad1.58x1.35mm_HandSolder -> Capacitors_SMD:C_0603; symbol trackix-rescue:C_Small-Device -> trackix-rescue:C_Small-Device-trackix-rescue
- C14: value 0,1uF -> 0.1uF; footprint Capacitor_SMD:C_0805_2012Metric_Pad1.15x1.40mm_HandSolder -> Capacitors_SMD:C_0603; symbol trackix-rescue:C_Small-Device -> trackix-rescue:C_Small-Device-trackix-rescue
- C15: value 22pF -> 10uF; footprint Capacitor_SMD:C_0805_2012Metric_Pad1.15x1.40mm_HandSolder -> Capacitors_SMD:C_1206; symbol trackix-rescue:C_Small-Device -> trackix-rescue:C_Small-Device-trackix-rescue
- C3: renamed from C?; value 0,1uF -> C_100nF; footprint Capacitor_SMD:C_0805_2012Metric_Pad1.15x1.40mm_HandSolder -> Capacitors_SMD:C_0603; symbol trackix-rescue:C_Small-Device -> trackix-rescue:C_Small-Device-trackix-rescue
- D2, D7, D8: footprint LEDs:LED_0805_HandSoldering -> LEDs:LED_0805; symbol trackix-rescue:LED-Device -> trackix-rescue:LED-Device-trackix-rescue
- D4, D5, D6: symbol trackix-rescue:LED-Device -> trackix-rescue:LED-Device-trackix-rescue
- IC2: footprint SOP-8 -> Housings_SOIC:HTSOP-8-1EP_3.9x4.9mm_Pitch1.27mm_ThermalVias_LargeCopper; symbol TP4056:TP4056 -> trackix-rescue:TP4056-TP4056-trackix-rescue
- J4: footprint Connector_PinSocket_2.54mm:PinSocket_2x03_P2.54mm_Vertical -> Socket_Strips:Socket_Strip_Straight_2x03_Pitch2.54mm_SMD; symbol trackix-rescue:AVR-ISP-6-Connector -> trackix-rescue:AVR-ISP-6-Connector-trackix-rescue
- Q1: footprint Package_TO_SOT_SMD:SOT-23_Handsoldering -> TO_SOT_Packages_SMD:SOT-23; symbol trackix-rescue:2N3904-Transistor_BJT -> trackix-rescue:2N3904-Transistor_BJT-trackix-rescue
- Q3: footprint SOP65P640X120-8N -> Housings_SSOP:TSSOP-8_4.4x3mm_Pitch0.65mm; symbol FS8205A:FS8205A -> trackix-rescue:FS8205A-FS8205A-trackix-rescue
- R1, R2: renamed from R?; footprint Resistors_SMD:R_0805_HandSoldering -> Resistors_SMD:R_0603; symbol trackix-rescue:R-Device -> trackix-rescue:R-Device-trackix-rescue
- R10, R11, R12, R7: value 470 -> 330; footprint Resistors_SMD:R_0805_HandSoldering -> Resistors_SMD:R_0603; symbol trackix-rescue:R-Device -> trackix-rescue:R-Device-trackix-rescue
- R13, R14, R15, R5, R6, R9: footprint Resistors_SMD:R_0805_HandSoldering -> Resistors_SMD:R_0603; symbol trackix-rescue:R-Device -> trackix-rescue:R-Device-trackix-rescue
- U1: footprint Package_QFP:TQFP-32_7x7mm_P0.8mm -> Housings_QFP:TQFP-32_7x7mm_Pitch0.8mm; symbol trackix-rescue:ATmega328P-AU-MCU_Microchip_ATmega -> trackix-rescue:ATmega328P-AU-MCU_Microchip_ATmega-trackix-rescue
- U3: footprint SOT23-6 -> TO_SOT_Packages_SMD:TSOT-23-6; symbol DW-01:DW-01 -> trackix-rescue:DW-01-DW-01-trackix-rescue
- reset1: symbol trackix-rescue:SW_Push-Switch -> trackix-rescue:SW_Push-Switch-trackix-rescue
Connections:
- net labels added: +3.3V, AUX_ON, CHARGE_DETECT, DIO_0, DIO_1, DIO_2, DRIVE_BUZZER, DRIVE_LED, GPS_TX, MISO, MOSI, NSS, RESET, RFM_RESET, SCK, SCL, SDA
- net labels removed: simRX, simTX
- wire segments 276 -> 302
Other:
- note added: "3.3v Regulator\n"
- note added: "ACCELEROMETER\n"
- note added: "BUZZER"
- note added: "Battery Charge + Protection"
- note added: "Decoupling VCC"
- note added: "MCU and programmer"
- note added: "MCU reset\n"
- note added: "RED LEDs\n"

Commit message: schematic ready for sim800L
Parts:
- removed C17: C_100nF, Capacitors_SMD:C_0603, symbol trackix-rescue:C_Small-Device-trackix-rescue
- removed J3: LORA_868, Connectors_Molex:Molex_Microcoaxial_RF, symbol trackix-rescue:Conn_Coaxial-Connector-trackix-rescue
- removed R21, R8: 4.7k, Resistors_SMD:R_0603, symbol trackix-rescue:R-Device-trackix-rescue
- removed U5: RFM95W-868S2, RF_Modules:Hopref_RFM9XW_SMD, symbol RF_Module:RFM95W-868S2
- removed U6: ADXL345BCCZ, Housings_LGA:Bosch_LGA-14_3x2.5mm_Pitch0.5mm, symbol ADXL345BCCZ:ADXL345BCCZ
- added J3: Conn_01x05_Male, Pin_Headers:Pin_Header_Straight_1x05_Pitch2.54mm, symbol Connector:Conn_01x05_Male
- added J5: Conn_01x05_Male, Pin_Headers:Pin_Header_Straight_1x05_Pitch2.54mm, symbol Connector:Conn_01x06_Male
- added JP2: PWR_BRIDGE, Jumper:SolderJumper-2_P1.3mm_Open_RoundedPad1.0x1.5mm, symbol Jumper:SolderJumper_2_Open
- added R3: R100, Resistors_SMD:R_0805, symbol device:R
- 8MHz1: footprint Crystals:Crystal_HC49-U_Vertical -> Crystals:Crystal_SMD_3225-4pin_3.2x2.5mm_HandSoldering
- C10, C11: footprint Capacitors_SMD:C_0402 -> Capacitors_SMD:C_0805
- C13: footprint Capacitors_SMD:C_0603 -> Capacitors_SMD:C_1206
- C14, C16, C3, C5, C7, C8: footprint Capacitors_SMD:C_0603 -> Capacitors_SMD:C_0805
- Q1, Q5: footprint TO_SOT_Packages_SMD:SOT-23 -> TO_SOT_Packages_SMD:SOT-23W_Handsoldering
- R1, R10, R11, R12, R13, R14, R15, R16, R17, R18, R19, R2, R20, R5, R6, R7, R9: footprint Resistors_SMD:R_0603 -> Resistors_SMD:R_0805
Connections:
- net +3V3: now also J3.5 (Pin_5), JP2.2 (B)
- net +BATT: now also JP2.1 (A)
- net GND: now also J3.1 (Pin_1); no longer U2.3 (RXD0)
- net DIO_0 renamed sim_ring
- net sim_ring: now also J5.1 (Pin_1)
- net DIO_1 renamed sim_dtr
- net sim_dtr: now also J5.2 (Pin_2)
- net DIO_2 renamed sim_rx
- net sim_rx: now also J3.2 (Pin_2)
- net NSS renamed sim_rst
- net sim_rst: now also J3.4 (Pin_4)
- net RFM_RESET renamed sim_tx
- net sim_tx: now also J3.3 (Pin_3)
- new net: R3.1, U2.3 (RXD0)
- new net GPS_RX: R3.2
Other:
- note added: "GPS RECEIVER"
- note added: "GSM networking SIM800L\n"
- note removed: "ACCELEROMETER\n"
- moved on the sheet: C12, C16, C4, C5, C6, C7, C9, D1, J2, L1, L2, R16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
